File: minipcie-breakout.kicad_pcb (KiCad board)
At the start: 2 copper layers, 33.3 x 65 mm, 5 parts, among them J2 Conn_01x26, J3 Conn_02x26_Odd_Even, J4 Conn_01x26

Commit message: latest version
Parts:
- added H3: MountingHole, MountingHole:MountingHole_2mm, F.Cu at (125.0, 100.0)
- added H4: MountingHole, MountingHole:MountingHole_2mm, F.Cu at (149.3, 100.0)
