File: minipcie-breakout.kicad_sch (KiCad schematic)
At the start: 5 parts, among them J2 Conn_01x26, J3 Conn_02x26_Odd_Even, J4 Conn_01x26

Commit message: latest version
Parts:
- added H3, H4: MountingHole, MountingHole:MountingHole_2mm, symbol Mechanical:MountingHole
Changed lines of the file:
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@@
 (kicad_sch
-	(version 20231120)
+	(version 20250114)
 	(generator "eeschema")
-	(generator_version "8.0")
+	(generator_version "9.0")
 	(paper "A4")
 	(text "total height:\nC426222 9.9mm \nC404125 9mm\nC2982553 8mm\nC367020 8mm\nC428485 7mm \nC428485 7mm\nC2761493 6.8mm\nC2761493 6.8mm \nC444927 5.2mm\nC185937 5.2mm\nC428488 4mm \nC266898 4mm\nC404119 4mm\n\n\n"
@@
 		)
 		(instances
-			(project ""
+			(project "minipcie-breakout"
 				(path "/8994f587-eb67-47f5-b451-806493e25754"
 					(reference "H2")
@@
 	)
 	(symbol
+		(lib_id "Mechanical:MountingHole")
+		(at 100.33 62.23 0)
+		(unit 1)
+		(exclude_from_sim yes)
+		(in_bom yes)
+		(on_board yes)
+		(dnp no)
+		(fields_autoplaced yes)
+		(property "Reference" "H4"
+			(at 102.87 60.9599 0)
+			(effects
+				(font
+					(size 1.27 1.27)
+				)
+				(justify left)
+			)
+		)
+		(property "Value" "MountingHole"
+			(at 102.87 63.4999 0)
+			(effects
+				(font
+					(size 1.27 1.27)
+				)
+				(justify left)
+			)
+		)
+		(property "Footprint" "MountingHole:MountingHole_2mm"
+			(at 100.33 62.23 0)
+			(effects
+				(font
+					(size 1.27 1.27)
+				)
+				(hide yes)
+			)
+		)
+		(property "Datasheet" "~"
+			(at 100.33 62.23 0)
+			(effects
+				(font
+					(size 1.27 1.27)
+				)
+				(hide yes)
+			)
+		)
+		(property "Description" "Mounting Hole without connection"
+			(at 100.33 62.23 0)
+			(effects
+				(font
+					(size 1.27 1.27)
+				)
+				(hide yes)
+			)
+		)
+		(property "LCSC" ""
+			(at 100.33 62.23 0)
+			(effects
+				(font
+					(size 1.27 1.27)
+				)
+				(hide yes)
+			)
+		)
+		(instances
+			(project "minipcie-breakout"
+				(path "/8994f587-eb67-47f5-b451-806493e25754"
+					(reference "H4")
+					(unit 1)
+				)
+			)
+		)
+	)
+	(symbol
 		(lib_id "Connector_Generic:Conn_02x27_Odd_Even")
 		(at 198.12 67.945 0)
@@
 				(path "/8994f587-eb67-47f5-b451-806493e25754"
 					(reference "J3")
+					(unit 1)
+				)
+			)
+		)
+	)
+	(symbol
+		(lib_id "Mechanical:MountingHole")
+		(at 100.33 55.88 0)
+		(unit 1)
+		(exclude_from_sim yes)
+		(in_bom yes)
+		(on_board yes)
+		(dnp no)
+		(fields_autoplaced yes)
+		(property "Reference" "H3"
+			(at 102.87 54.6099 0)
+			(effects
+				(font
+					(size 1.27 1.27)
+				)
+				(justify left)
+			)
+		)
+		(property "Value" "MountingHole"
+			(at 102.87 57.1499 0)
+			(effects
+				(font
+					(size 1.27 1.27)
+				)
+				(justify left)
+			)
+		)
+		(property "Footprint" "MountingHole:MountingHole_2mm"
+			(at 100.33 55.88 0)
+			(effects
+				(font
+					(size 1.27 1.27)
+				)
+				(hide yes)
+			)
+		)
+		(property "Datasheet" "~"
+			(at 100.33 55.88 0)
+			(effects
+				(font
+					(size 1.27 1.27)
+				)
+				(hide yes)
+			)
+		)
+		(property "Description" "Mounting Hole without connection"
+			(at 100.33 55.88 0)
+			(effects
+				(font
+					(size 1.27 1.27)
+				)
+				(hide yes)
+			)
+		)
+		(property "LCSC" ""
+			(at 100.33 55.88 0)
+			(effects
+				(font
+					(size 1.27 1.27)
+				)
+				(hide yes)
+			)
+		)
+		(instances
+			(project "minipcie-breakout"
+				(path "/8994f587-eb67-47f5-b451-806493e25754"
+					(reference "H3")
 					(unit 1)
 				)
@@
 		)
 		(instances
-			(project ""
+			(project "minipcie-breakout"
 				(path "/8994f587-eb67-47f5-b451-806493e25754"
 					(reference "H1")
@@
 		)
 	)
+	(embedded_fonts no)
 )
